File: emrelabs-PanelDuino-2x8.brd (EAGLE design)
At the start: 90 x 45 mm, 64 parts, among them CN1 USB-MICROB, CN11 AVR-ICSP, U1 7805, U3 CH340G, U4 PCF8574, U5 ATMEGA328PA, U6 PCF8574

Commit message: Crystal value updated
Parts:
- XT2: value 8MHz -> 16Mhz
Changed lines of the file:
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@@
 <drawing>
 <settings>
-<setting alwaysvectorfont="yes"/>
+<setting alwaysvectorfont="no"/>
 <setting keepoldvectorfont="yes"/>
 <setting verticaltext="up"/>
@@
 <attribute name="MANUFACTURER" value="" x="44.75" y="-14.75" size="1.778" layer="27" rot="R90" display="off"/>
 </element>
-<element name="XT2" library="Elib-RLC-D-XT" package="XT-HC49" value="8MHz" x="52" y="22.5" rot="R90"/>
+<element name="XT2" library="Elib-RLC-D-XT" package="XT-HC49" value="16Mhz" x="52" y="22.5" rot="R90"/>
 <element name="C28" library="Elib-RLC-D-XT" package="C1206" value="100n" x="68.5" y="14.75" rot="R270">
 <attribute name="DIGIKEYPN" value="" x="80.5" y="49.75" size="1.778" layer="27" rot="R270" display="off"/>
